Commit message: Update work version of twolink scene

File: exoskeleton_description/urdf/exo.gazebo.xacro (robot description, xacro)
@@ -1,5 +1,4 @@
 <?xml version="1.0"?>
-<robot xmlns:xacro="http://www.ros.org/wiki/xacro"
-      xmlns:sensor="http://playerstage.sourceforge.net/gazebo/xmlschema/#sensor">
+<robot xmlns:xacro="http://www.ros.org/wiki/xacro">
   <xacro:macro name="exo_gazebo" params="robot_name">
     <gazebo>

File: exoskeleton_description/urdf/exo.transmission.xacro (robot description, xacro)
@@ -1,5 +1,5 @@
 <?xml version="1.0"?>
 <robot xmlns:xacro="http://www.ros.org/wiki/xacro">
-  <xacro:macro name="exo_transmission" params="hardware_interface">
+  <xacro:macro name="exo_transmission" params="hardware_interface robot_name">
     <transmission name="${robot_name}_tran_1">
       <robotNamespace>/${robot_name}</robotNamespace>

File: exoskeleton_description/urdf/exo_left.urdf.xacro (robot description, xacro)
@@ -12,3 +12,6 @@
     <origin xyz="$(arg origin_xyz)" rpy="$(arg origin_rpy)" />
   </xacro:exo_left>
+  <!-- <xacro:exo_left hardware_interface="$(arg hardware_interface)" robot_name="exo2" parent="world">
+    <origin xyz="1 0 2" rpy="$(arg origin_rpy)" />
+  </xacro:exo_left> -->
 </robot>

File: exoskeleton_description/urdf/exo_left.xacro (robot description, xacro)
@@ -35,9 +35,16 @@
             filename="package://exoskeleton_description/meshes/base_short.stl"
             scale="0.01 0.01 0.01" />
-          <material>
-            <color rgba="1 0 0 1" />
-          </material>
         </geometry>
+<material name="Grey"/>
       </visual>
+      <!-- <collision>
+        <origin xyz="-0.1 -0.05 -0.05" rpy="0 0 0" />
+        <geometry>
+          <mesh
+            filename="package://exoskeleton_description/meshes/base_short.stl"
+            scale="0.01 0.01 0.01" />
+        </geometry>
+<material name="Grey"/>
+      </collision> -->
     </link>
     <joint name="${robot_name}_joint_1" type="revolute">
@@ -72,9 +79,16 @@
             filename="package://exoskeleton_description/meshes/link.stl"
             scale="0.01 0.01 0.01" />
-          <material>
-            <color rgba="0 1 0 1" />
-          </material>
         </geometry>
+<material name="Grey"/>
       </visual>
+      <!-- <collision>
+        <origin xyz="0.1 -0.05 -0.05" rpy="0 0 0" />
+        <geometry>
+          <mesh
+            filename="package://exoskeleton_description/meshes/link.stl"
+            scale="0.01 0.01 0.01" />
+        </geometry>
+<material name="Grey"/>
+      </collision> -->
     </link>
     <joint name="${robot_name}_joint_2" type="revolute">
@@ -109,13 +123,20 @@
             filename="package://exoskeleton_description/meshes/link.stl"
             scale="0.01 0.01 0.01" />
-          <material>
-            <color rgba="0 0 1 1" />
-          </material>
         </geometry>
+<material name="Grey"/>
       </visual>
+      <!-- <collision>
+        <origin xyz="0.05 -0.05 0" rpy="0 0 0" />
+        <geometry>
+          <mesh
+            filename="package://exoskeleton_description/meshes/link.stl"
+            scale="0.01 0.01 0.01" />
+        </geometry>
+<material name="Grey"/>
+      </collision> -->
     </link>
     <!--Extensions -->
     <xacro:exo_gazebo robot_name="${robot_name}" />
-    <xacro:exo_transmission hardware_interface="${hardware_interface}"/>
+    <xacro:exo_transmission hardware_interface="${hardware_interface}" robot_name="$(arg robot_name)"/>
   </xacro:macro>
 </robot>
